File: VFO_80289.kicad_sch (KiCad schematic)
At the start: 96 parts, among them Q89-1 2N5486, Q89-2 MPS6514, Q89-3 2N5486, Q89-4 MPS6514, Q89-5 MPS6512, U89-1 MC1496P, Y89-1 7.5MHz, Y89-2 11MHz, Y89-3 6.99MHz

Commit message: Release VFO 80289 and mixer 80287 v0.2.0
Parts:
- added R89-89: 50, symbol Device:R_Small_US
- added V89-1: 13.8, symbol Simulation_SPICE:VDC
- added V89-2: 8.0, symbol Simulation_SPICE:VDC
- added V89-3: 3.1, symbol Simulation_SPICE:VDC
- C89-10: value 5-60p -> {VFO_C10}
- C89-11: value 5-60p -> {VFO_C11}
- C89-12: value 5-60p -> {VFO_C12}
- C89-13, C89-14, C89-15: value .01 -> .01u
- C89-35: value Selected in production -> 3p
- C89-7: value 5-60p -> {VFO_C7}
- C89-8: value 5-60p -> {VFO_C8}
- C89-9: value 5-60p -> {VFO_C9}
- L89-101: value L_Trim -> {VFO_T1_L1}
- L89-102: value L_Trim -> {VFO_T1_L2}
Connections:
- net +12: now also V89-1.1
- net +REG: now also V89-2.1
- net GND: now also R89-89.2, V89-1.2, V89-2.2, V89-3.2
- net OFFSET: now also V89-3.1
- net OUT: now also R89-89.1
Other:
- note added: "* VFO magnetic, trimmer, and alignment-control values below are inferred simulation-aligned values, not factory specifications .param PTO_L1=0.8u .param PTO_L2=10u .param PTO_L3=13u .param VFO_R2_POS=0.760 .param VFO_R27_POS=0.100 .param VFO_T1_L1=5.221u .param VFO_T1_L2=4.567u .param VFO_T1_K=0.2463 .param VFO_C7=25.73p .param VFO_C8=6.697p .param VFO_C9=31.28p .param VFO_C10=20.35p .param VFO_C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"
