File: VFO_80289.kicad_sch (KiCad schematic)
At the start: 100 parts, among them Q89-1 2N5486, Q89-2 MPS6514, Q89-3 2N5486, Q89-4 MPS6514, Q89-5 MPS6512, U89-1 MC1496P, Y89-1 7.5MHz, Y89-2 11MHz, Y89-3 6.99MHz

Commit message: Complete IF-AGC schematic and SPICE models
Parts:
- renumbered L1 to L89-5
Other:
- company: Andy McCann KA3KAF & DOug McCann KA3KAG -> Andy McCann KA3KAF & Doug McCann KA3KAG
Changed lines of the file:
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@@
 		(date "2026-07-26")
 		(rev "0.2")
-		(company "Andy McCann KA3KAF & DOug McCann KA3KAG")
-		(comment 2 "Original Design: Ten-Tec")
-		(comment 3 "Triton IV (Model 540)")
+		(company "Andy McCann KA3KAF & Doug McCann KA3KAG")
+		(comment 3 "Seveirville TN")
+		(comment 4 "Original Design: Ten-Tec")
+		(comment 5 "Triton IV (Model 540)")
 	)
 	(rectangle
@@
 		(dnp no)
 		(fields_autoplaced yes)
-		(property "Reference" "L1"
+		(property "Reference" "L89-5"
 			(at 116.84 207.0099 0)
 			(show_name no)
@@
 			(project "triton_540"
 				(path "/2d45daab-5f60-4e97-8c02-32b0054eab28/818ce5bb-55e6-4013-915b-e8afd4640f1a"
-					(reference "L1")
+					(reference "L89-5")
 					(unit 1)
 				)
