File: RF_Amp_80166.kicad_sch (KiCad schematic)
At the start: 18 parts, among them Q66-1 40823, T66-1 9MHz Trap

Commit message: Release VFO 80289 and mixer 80287 v0.2.0
Parts:
- added C66-101: 5p, symbol Device:C_Small_US
- added R66-100: 1Meg, symbol Device:R_Small_US
- added R66-99: 50, symbol Device:R_Small_US
- added V66-1: 3.9, symbol Simulation_SPICE:VDC
- added V66-2: 12, symbol Simulation_SPICE:VDC
- added V7: 0, symbol Simulation_SPICE:VDC
Connections:
- net ANT: now also R66-99.2
- net DEFEAT: now also V66-1.1
- net GND: now also C66-101.2, R66-100.1, V66-1.2, V66-2.2, V7.2
- net R: now also V66-2.1
- new net: C66-101.1, R66-100.2
- new net: R66-99.1, V7.1
Other:
- note added: ".option rshunt=1e12"
- note added: ".param L_RACK=1.4253u .param L2_TRACK=0.0849053 .param L2_OFFSET=1.97963u"
- note added: "L_RACK represents the RESONATE-control position"

Commit message: Complete IF-AGC schematic and SPICE models
Other:
- company: Andy McCann KA3KAF & DOug McCann KA3KAG -> Andy McCann KA3KAF & Doug McCann KA3KAG
Changed lines of the file:
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@@
 		(date "2026-07-26")
 		(rev "0.2")
-		(company "Andy McCann KA3KAF & DOug McCann KA3KAG")
-		(comment 2 "Original Design: Ten-Tec")
-		(comment 3 "Triton IV (Model 540)")
+		(company "Andy McCann KA3KAF & Doug McCann KA3KAG")
+		(comment 3 "Seveirville TN")
+		(comment 4 "Original Design: Ten-Tec")
+		(comment 5 "Triton IV (Model 540)")
 	)
 	(rectangle
