File: tx_rx_mixer_80287.kicad_sch (KiCad schematic)
At the start: 45 parts, among them U87-1 MC1496P, U87-2 MC1496P

Commit message: Add TX-RX mixer simulations
Parts:
- added C87-18: 22p, symbol Device:C_Small_US
- added R87-90: 10k, symbol Device:R_Small_US
- added R87-91: 50, symbol Device:R_Small_US
- added V87-1: .6, symbol Simulation_SPICE:VDC
- added V87-2: 10.4, symbol Simulation_SPICE:VDC
- added V87-3, V87-4, V87-5, V87-6: 1, symbol Simulation_SPICE:VSIN
- C87-14: value 100u -> 100p
- L87-1: value L_Iron_Small -> 1u
- L87-2: renamed from L2; value L_Small_Center_Tap -> 10u/half estimated
- L87-3: value L_Trim -> ${SIM.PARAMS}
Connections:
- net GND: now also R87-90.2, R87-91.2, V87-1.2, V87-2.2, V87-3.2, V87-4.2, V87-5.2, V87-6.2
- net OUT: now also R87-91.1
- net R: now also V87-1.1
- net Rx 9MHz: now also R87-90.1
- net Rx In: now also C87-1.1, V87-3.1
- net T: now also V87-2.1
- net Tx 9MHz: now also V87-5.1
- net Tx VFO: now also C87-18.2, V87-6.1; no longer C87-15.2, C87-17.1, L87-1.1
- net at C87-5.1, C87-8.1, D87-1.1 (K)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: now also C87-20.2, C87-6.1, R87-3.1, R87-4.2
- net at R87-6.1, R87-7.2: now also C87-3.2, R87-5.1, U87-1.10 (Carrier_Input)
- net Rx VFO  renamed Rx VFO
- net Rx VFO: now also V87-4.1
- new net: C87-15.2, C87-17.1, C87-18.1, L87-1.1

Commit message: Complete IF-AGC schematic and SPICE models
Other:
- company: Andy McCann KA3KAF & DOug McCann KA3KAG -> Andy McCann KA3KAF & Doug McCann KA3KAG
Changed lines of the file:
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@@
 		(date "2026-07-26")
 		(rev "0.2")
-		(company "Andy McCann KA3KAF & DOug McCann KA3KAG")
-		(comment 2 "Original Design: Ten-Tec")
-		(comment 3 "Triton IV (Model 540)")
+		(company "Andy McCann KA3KAF & Doug McCann KA3KAG")
+		(comment 3 "Seveirville TN")
+		(comment 4 "Original Design: Ten-Tec")
+		(comment 5 "Triton IV (Model 540)")
 	)
 	(rectangle
