File: 80166_rf_amp.kicad_sch (KiCad schematic)
At the start: 24 parts, among them Q66-1 40823, T66-1 9MHz Trap

Commit message: Repair and re-enable 80166 simulation in the shared schematic
A fresh SPICE export contained no 80166 nets at all, and three separate faults
had accumulated during later work on the other assemblies. All three are
simulation-only; none of them affects the reconstruction of the circuit.

Sheet selection. The root schematic can only usefully simulate one assembly at
a time. RF_Amp_80166 is now included and IF-AGC_80279, VFO-80289 and
TX RX Mixer 80287 are excluded. Running a study for one of those boards means
reversing this. exclude_from_sim was also switched off on the 80166 sub-sheet's
test fixture (V7, R66-99, R66-100, C66-101, V66-1, V66-2) and on the off-board
bandswitch parts the tuned circuits need (S4, S4B1, C8-C20).

S4B1's SPICE pin map. The bandswitch is one physical rotary switch with two
wafers, drawn as two units of triton_iv:SW_Rotary_1x5_multiunit. When that
library symbol was reworked, unit 2's pins were renumbered 7-12, but S4B1's
Sim.Pins property still mapped the model's terminals to symbol pins 1-6, which
belong to unit 1. KiCad exported the switch with every terminal unconnected, so
the entire L2 tuning network -- C13 through C20 -- hung off nothing and the
output tuned circuit could not resonate. Sim.Pins now reads 7=1 8=2 ... 12=6.

A missing OUT label. The simulation-fixture area of the 80166 sub-sheet had no
local OUT label, so the provisional 1 MOhm || 5 pF output load sat on an
unnamed net instead of on the OUT pin. The load was floating.

Verified against the retained evidence after the repairs: the 29 MHz aligned
peak comes back at 28.999790 MHz against the retained 28.999365 MHz, which is
within one 0.45 kHz sweep step; Q1's source voltage and drain current reproduce
Simulation 1 exactly at 2.071 V and 4.407 mA; and the 3.500 MHz peak gain
reproduces Simulation 2 exactly at 20.189 dB. ERC reports the same 61
violations before and after, identical by type.

One naming consequence, which invalidates no evidence. The ANT and OUT pins are
w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
Connections:
- net OUT: now also C66-101.1, R66-100.2
Changed lines of the file:
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@@
 		)
 	)
+	(label "OUT"
+		(at 100.33 168.91 0)
+		(effects
+			(font
+				(size 1.27 1.27)
+			)
+			(justify left bottom)
+		)
+	)
 	(label "ANT"
 		(at 83.82 167.64 0)
@@
 		(unit 1)
 		(body_style 1)
-		(exclude_from_sim yes)
+		(exclude_from_sim no)
 		(in_bom yes)
 		(on_board yes)
@@
 		(unit 1)
 		(body_style 1)
-		(exclude_from_sim yes)
+		(exclude_from_sim no)
 		(in_bom yes)
 		(on_board yes)
@@
 		(unit 1)
 		(body_style 1)
-		(exclude_from_sim yes)
+		(exclude_from_sim no)
 		(in_bom yes)
 		(on_board yes)
@@
 		(unit 1)
 		(body_style 1)
-		(exclude_from_sim yes)
+		(exclude_from_sim no)
 		(in_bom yes)
 		(on_board yes)
@@
 		(unit 1)
 		(body_style 1)
-		(exclude_from_sim yes)
+		(exclude_from_sim no)
 		(in_bom yes)
 		(on_board yes)
@@
 		(unit 1)
 		(body_style 1)
-		(exclude_from_sim yes)
+		(exclude_from_sim no)
 		(in_bom yes)
 		(on_board yes)
@@
 		(unit 1)
 		(body_style 1)
-		(exclude_from_sim yes)
+		(exclude_from_sim no)
 		(in_bom yes)
 		(on_board yes)
@@
 		(unit 1)
 		(body_style 1)
-		(exclude_from_sim yes)
+		(exclude_from_sim no)
 		(in_bom yes)
 		(on_board yes)
@@
 		(unit 1)
 		(body_style 1)
-		(exclude_from_sim yes)
+		(exclude_from_sim no)
 		(in_bom yes)
 		(on_board yes)
@@
 		(unit 1)
 		(body_style 1)
-		(exclude_from_sim yes)
+		(exclude_from_sim no)
 		(in_bom yes)
 		(on_board yes)
@@
 		(unit 1)
 		(body_style 1)
-		(exclude_from_sim yes)
+		(exclude_from_sim no)
 		(in_bom yes)
 		(on_board yes)
